File: minilab/ml-hardware/oscillator.kicad_sch (KiCad schematic)
At the start: 6 parts, among them U2 NE555P

Commit message: minilab: Enforce "pcb/page" hierarchy on schematic
This does not apply (necessarily) to subpages.
Parts:
- C9: footprint (none) -> Capacitor_THT:C_Disc_D6.0mm_W2.5mm_P5.00mm
- D2: renamed from D7; footprint (none) -> LED_THT:LED_Rectangular_W5.0mm_H2.0mm
- R18: renamed from R21; footprint (none) -> Resistor_THT:R_Axial_DIN0204_L3.6mm_D1.6mm_P5.08mm_Horizontal
- R19: renamed from R22; footprint (none) -> Resistor_THT:R_Axial_DIN0204_L3.6mm_D1.6mm_P5.08mm_Horizontal
- RV1: footprint (none) -> Potentiometer_THT:Potentiometer_Bourns_3296W_Vertical
Changed lines of the file:
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@@
 		(dnp no)
 		(fields_autoplaced yes)
-		(property "Reference" "D7"
+		(property "Reference" "D2"
 			(at 180.34 99.3774 90)
 			(effects
@@
 			)
 		)
-		(property "Footprint" ""
+		(property "Footprint" "LED_THT:LED_Rectangular_W5.0mm_H2.0mm"
 			(at 176.53 99.06 0)
 			(effects
@@
 		)
 		(instances
-			(project ""
-				(path "/edb8a0df-1def-48df-b494-4a6b89ce8f9c/cee87e4e-7aee-4a91-91ad-8832d36e7e19"
-					(reference "D7")
+			(project "ml-hardware"
+				(path "/edb8a0df-1def-48df-b494-4a6b89ce8f9c/d397cdb8-1135-4612-aff9-bdf84d932419/bc259005-a59b-4e7b-a399-bea54a015299"
+					(reference "D2")
 					(unit 1)
 				)
@@
 			)
 		)
-		(property "Footprint" ""
+		(property "Footprint" "Potentiometer_THT:Potentiometer_Bourns_3296W_Vertical"
 			(at 152.4 99.06 0)
 			(effects
@@
 		(instances
 			(project "ml-hardware"
-				(path "/edb8a0df-1def-48df-b494-4a6b89ce8f9c/cee87e4e-7aee-4a91-91ad-8832d36e7e19"
+				(path "/edb8a0df-1def-48df-b494-4a6b89ce8f9c/d397cdb8-1135-4612-aff9-bdf84d932419/bc259005-a59b-4e7b-a399-bea54a015299"
 					(reference "RV1")
 					(unit 1)
@@
 		(dnp no)
 		(fields_autoplaced yes)
-		(property "Reference" "R21"
+		(property "Reference" "R18"
 			(at 154.94 80.0099 0)
 			(effects
@@
 			)
 		)
-		(property "Footprint" ""
+		(property "Footprint" "Resistor_THT:R_Axial_DIN0204_L3.6mm_D1.6mm_P5.08mm_Horizontal"
 			(at 150.622 81.28 90)
 			(effects
@@
 		)
 		(instances
-			(project ""
-				(path "/edb8a0df-1def-48df-b494-4a6b89ce8f9c/cee87e4e-7aee-4a91-91ad-8832d36e7e19"
-					(reference "R21")
+			(project "ml-hardware"
+				(path "/edb8a0df-1def-48df-b494-4a6b89ce8f9c/d397cdb8-1135-4612-aff9-bdf84d932419/bc259005-a59b-4e7b-a399-bea54a015299"
+					(reference "R18")
 					(unit 1)
 				)
@@
 			)
 		)
-		(property "Footprint" ""
+		(property "Footprint" "Capacitor_THT:C_Disc_D6.0mm_W2.5mm_P5.00mm"
 			(at 153.3652 116.84 0)
 			(effects
@@
 		)
 		(instances
-			(project ""
-				(path "/edb8a0df-1def-48df-b494-4a6b89ce8f9c/cee87e4e-7aee-4a91-91ad-8832d36e7e19"
+			(project "ml-hardware"
+				(path "/edb8a0df-1def-48df-b494-4a6b89ce8f9c/d397cdb8-1135-4612-aff9-bdf84d932419/bc259005-a59b-4e7b-a399-bea54a015299"
 					(reference "C9")
 					(unit 1)
@@
 		(instances
 			(project "ml-hardware"
-				(path "/edb8a0df-1def-48df-b494-4a6b89ce8f9c/cee87e4e-7aee-4a91-91ad-8832d36e7e19"
+				(path "/edb8a0df-1def-48df-b494-4a6b89ce8f9c/d397cdb8-1135-4612-aff9-bdf84d932419/bc259005-a59b-4e7b-a399-bea54a015299"
 					(reference "U2")
 					(unit 1)
@@
 		(dnp no)
 		(fields_autoplaced yes)
-		(property "Reference" "R22"
+		(property "Reference" "R19"
 			(at 179.07 111.7599 0)
 			(effects
@@
 			)
 		)
-		(property "Footprint" ""
+		(property "Footprint" "Resistor_THT:R_Axial_DIN0204_L3.6mm_D1.6mm_P5.08mm_Horizontal"
 			(at 174.752 113.03 90)
 			(effects
@@
 		(instances
 			(project "ml-hardware"
-				(path "/edb8a0df-1def-48df-b494-4a6b89ce8f9c/cee87e4e-7aee-4a91-91ad-8832d36e7e19"
-					(reference "R22")
-					(unit 1)
-				)
+				(path "/edb8a0df-1def-48df-b494-4a6b89ce8f9c/d397cdb8-1135-4612-aff9-bdf84d932419/bc259005-a59b-4e7b-a399-bea54a015299"
+					(reference "R19")
+					(unit 1)
+				)

Commit message: minilab: cambia jerarquia y agrega pcb
Parts:
- added C10: 10nF, Capacitor_THT:C_Disc_D6.0mm_W2.5mm_P5.00mm, symbol Device:C
- U2: footprint Package_DIP:DIP-8_W7.62mm -> Package_DIP:DIP-8_W7.62mm_LongPads
Connections:
- net GND: now also C10.2
- net at C9.1, RV1.3, U2.2 (TR): now also U2.6 (THR)
- net at U2.5 (CV): now also C10.1
- no-connect marks 2 -> 0
Changed lines of the file:
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@@
+	)
+	(junction
+		(at 144.78 105.41)
+		(diameter 0)
+		(color 0 0 0 0)
 	)
 	(junction
@@
 		(color 0 0 0 0)
 	)
-	(no_connect
-		(at 116.84 92.71)
-	)
-	(no_connect
-		(at 142.24 97.79)
+	(wire
+		(pts
+			(xy 100.33 95.25) (xy 100.33 92.71)
+		)
+		(stroke
+			(width 0)
+			(type default)
+		)
 	)
 	(wire
@@
 	(wire
 		(pts
+			(xy 144.78 105.41) (xy 152.4 105.41)
+		)
+		(stroke
+			(width 0)
+			(type default)
+		)
+	)
+	(wire
+		(pts
 			(xy 176.53 95.25) (xy 176.53 87.63)
 		)
@@
 	(wire
 		(pts
+			(xy 100.33 92.71) (xy 116.84 92.71)
+		)
+		(stroke
+			(width 0)
+			(type default)
+		)
+	)
+	(wire
+		(pts
 			(xy 147.32 99.06) (xy 147.32 92.71)
 		)
@@
 	(wire
 		(pts
+			(xy 100.33 102.87) (xy 100.33 120.65)
+		)
+		(stroke
+			(width 0)
+			(type default)
+		)
+	)
+	(wire
+		(pts
+			(xy 144.78 97.79) (xy 144.78 105.41)
+		)
+		(stroke
+			(width 0)
+			(type default)
+		)
+	)
+	(wire
+		(pts
 			(xy 152.4 92.71) (xy 152.4 95.25)
 		)
@@
 	(wire
 		(pts
+			(xy 142.24 97.79) (xy 144.78 97.79)
+		)
+		(stroke
+			(width 0)
+			(type default)
+		)
+	)
+	(wire
+		(pts
 			(xy 152.4 102.87) (xy 152.4 105.41)
 		)
@@
 	(wire
 		(pts
-			(xy 111.76 105.41) (xy 152.4 105.41)
+			(xy 111.76 105.41) (xy 144.78 105.41)
 		)
 		(stroke
@@
 		(shape input)
 		(at 152.4 120.65 270)
+		(effects
+			(font
+				(size 1.27 1.27)
+			)
+			(justify right)
+		)
+	)
+	(hierarchical_label "GND"
+		(shape input)
+		(at 100.33 120.65 270)
 		(effects
 			(font
@@
 			)
 		)
-		(property "Footprint" "Package_DIP:DIP-8_W7.62mm"
+		(property "Footprint" "Package_DIP:DIP-8_W7.62mm_LongPads"
 			(at 146.05 102.87 0)
 			(effects
@@
 					(unit 1)
 				)
+			)
+		)
+	)
+	(symbol
+		(lib_id "Device:C")
+		(at 100.33 99.06 0)
+		(unit 1)
+		(exclude_from_sim no)
+		(in_bom yes)
+		(on_board yes)
+		(dnp no)
+		(fields_autoplaced yes)
+		(property "Reference" "C10"
+			(at 104.14 97.7899 0)
+			(effects
+				(font
+					(size 1.27 1.27)
+				)
+				(justify left)
+			)
+		)
+		(property "Value" "10nF"
+			(at 104.14 100.3299 0)
+			(effects
+				(font
+					(size 1.27 1.27)
+				)
+				(justify left)
+			)
+		)
+		(property "Footprint" "Capacitor_THT:C_Disc_D6.0mm_W2.5mm_P5.00mm"
+			(at 101.2952 102.87 0)
+			(effects
+				(font
+					(size 1.27 1.27)
+				)
+				(hide yes)
+			)
+		)
+		(property "Datasheet" "~"
+			(at 100.33 99.06 0)
+			(effects
+				(font
+					(size 1.27 1.27)
+				)
+				(hide yes)
+			)
+		)
+		(property "Description" "Unpolarized capacitor"
+			(at 100.33 99.06 0)
+			(effects
+				(font
+					(size 1.27 1.27)
+				)
+				(hide yes)
+			)
+		)
+		(pin "2"
+		)
+		(pin "1"
+		)
+		(instances
+			(project "ml-hardware"
+				(path "/edb8a0df-1def-48df-b494-4a6b89ce8f9c/d397cdb8-1135-4612-aff9-bdf84d932419/bc259005-a59b-4e7b-a399-bea54a015299"
+					(reference "C10")
+					(unit 1)
+				)
